File: nsc-v2.1/ns-clock-neo/ns-clock-neo.kicad_pcb (KiCad board)
At the start: 2 copper layers, 43.7 x 46.5 mm, 12 parts, among them J2 Bat connector, J3 Conn_01x14_Pin, J4 Conn_01x14_Pin, J5 Bat connector, J6 Conn_01x14_Pin, J7 Conn_01x14_Pin, U1 2764, U4 2764, Y1 32.768 kHz, Y2 32.768 kHz

Commit message: Add files via upload
Routing:
- net +5V: track 98.5 -> 101.1 mm
- net CE: track 34.1 -> 35.2 mm, vias 1 -> 3
- net GND: track 66.9 -> 68.0 mm
Changed lines of the file:
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@@
-	)
-	(segment
-		(start 106.68 80.01)
-		(end 104.14 77.47)
-		(width 0.2)
-		(layer "B.Cu")
-		(net "GND")
-	)
-	(segment
-		(start 106.68 85.09)
-		(end 106.68 80.01)
-		(width 0.2)
-		(layer "B.Cu")
-		(net "GND")
 	)
 	(segment
@@
 	)
 	(segment
+		(start 109.22 85.09)
+		(end 104.14 80.01)
+		(width 0.2)
+		(layer "B.Cu")
+		(net "GND")
+	)
+	(segment
+		(start 104.14 80.01)
+		(end 104.14 77.47)
+		(width 0.2)
+		(layer "B.Cu")
+		(net "GND")
+	)
+	(segment
 		(start 136.93 85.06)
 		(end 134.39 85.06)
@@
 	)
 	(segment
-		(start 112.99 83.78)
+		(start 106.68 83.78)
 		(end 97.83 83.78)
 		(width 0.2)
@@
 	)
 	(segment
+		(start 126.77 40.584)
+		(end 126.746 40.56)
+		(width 0.2)
+		(layer "F.Cu")
+		(net "+5V")
+	)
+	(segment
 		(start 113.255 84.045)
 		(end 114.3 85.09)
@@
 	)
 	(segment
+		(start 106.68 85.09)
+		(end 106.68 83.78)
+		(width 0.2)
+		(layer "F.Cu")
+		(net "+5V")
+	)
+	(segment
+		(start 120.47 40.56)
+		(end 126.746 40.56)
+		(width 0.2)
+		(layer "F.Cu")
+		(net "+5V")
+	)
+	(segment
+		(start 112.99 83.78)
+		(end 106.68 83.78)
+		(width 0.2)
+		(layer "F.Cu")
+		(net "+5V")
+	)
+	(segment
+		(start 126.77 41.88)
+		(end 126.77 40.584)
+		(width 0.2)
+		(layer "F.Cu")
+		(net "+5V")
+	)
+	(segment
 		(start 136.93 41.88)
 		(end 135.66 43.15)
@@
 	)
 	(segment
-		(start 120.47 40.56)
+		(start 126.746 40.56)
 		(end 135.61 40.56)
 		(width 0.2)
@@
 	(segment
 		(start 99.06 83.03)
-		(end 99.06 82.55)
-		(width 0.2)
-		(layer "F.Cu")
-		(net "CE")
-	)
-	(segment
-		(start 99.06 82.55)
-		(end 100.33 81.28)
-		(width 0.2)
-		(layer "F.Cu")
-		(net "CE")
-	)
-	(segment
-		(start 109.474 81.28)
-		(end 110.49 80.264)
+		(end 99.088 83.058)
 		(width 0.2)
 		(layer "F.Cu")
@@
 	)
 	(segment
+		(start 99.088 83.058)
+		(end 108.331 83.058)
+		(width 0.2)
+		(layer "F.Cu")
+		(net "CE")
+	)
+	(segment
+		(start 110.49 78.613)
+		(end 110.49 74.93)
+		(width 0.2)
+		(layer "F.Cu")
+		(net "CE")
+	)
+	(segment
 		(start 109.728 74.168)
 		(end 109.728 64.262)
@@
 		(net "CE")
 	)
-	(segment
-		(start 110.49 80.264)
-		(end 110.49 74.93)
-		(width 0.2)
-		(layer "F.Cu")
-		(net "CE")
-	)
-	(segment
-		(start 100.33 81.28)
-		(end 109.474 81.28)
-		(width 0.2)
-		(layer "F.Cu")
+	(via
+		(at 108.331 83.058)
+		(size 0.6)
+		(drill 0.3)
+		(layers "F.Cu" "B.Cu")
 		(net "CE")
 	)
@@
 		(net "CE")
 	)
+	(via
+		(at 110.49 78.613)
+		(size 0.6)
+		(drill 0.3)
+		(layers "F.Cu" "B.Cu")
+		(net "CE")
+	)
+	(segment
+		(start 109.982 83.058)
+		(end 110.49 82.55)
+		(width 0.2)
+		(layer "B.Cu")
+		(net "CE")
+	)
 	(segment
 		(start 99.06 83.03)
@@
 		(width 0.2)
 		(layer "B.Cu")
+		(net "CE")
+	)
+	(segment
+		(start 110.49 82.55)
+		(end 110.49 78.613)
+		(width 0.2)
+		(layer "B.Cu")
+		(net "CE")
+	)
+	(segment
+		(start 108.331 83.058)
+		(end 109.982 83.058)
+		(width 0.2)
+		(layer "B.Cu")
