File: nsc-v3/ns-clock-neo/ns-clock-neo.kicad_pcb (KiCad board)
At the start: 2 copper layers, 26.3 x 82.5 mm, 6 parts, among them J2 Bat connector, J3 Conn_01x14_Pin, J4 Conn_01x14_Pin, U1 2764, Y1 32.768 kHz

Commit message: Add files via upload
Parts:
- moved J3 36.4 mm to (114.3, 76.2), turned to 180 degrees
- moved J4 36.4 mm to (99.1, 76.2), turned to 180 degrees
- moved U1 34.1 mm to (114.3, 91.4), turned to 180 degrees
- moved DS1215 1.80 mm to (114.3, 87.6)
- renumbered U2 to DS1215
Routing:
- net +5V: track 143.0 -> 39.1 mm
- net D0: track 41.4 -> 142.7 mm
- net D2: track 19.9 -> 112.9 mm
- net D1: track 25.3 -> 107.6 mm
- net D3: track 15.5 -> 88.2 mm
- net A0: track 50.4 -> 122.9 mm, vias 0 -> 2
- net VPP: track 84.7 -> 16.4 mm
- net D4: track 19.9 -> 82.7 mm
- net A12: track 77.1 -> 21.5 mm
- net PGM: track 77.0 -> 23.8 mm
- net D5: track 25.3 -> 77.2 mm
- net A1: track 41.5 -> 90.1 mm
- net D6: track 30.7 -> 71.8 mm
- net A2: track 74.3 -> 108.1 mm
- net A8: track 66.5 -> 34.3 mm
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Other:
- board size 26.3 x 82.5 mm -> 26.7 x 85.3 mm
- board text added: "- BAT +"
- board text added: "04/06/2026"
- board text added: "Plug this in ROM CD or MON Socket"
- board text added: "no slot clock neo"
- board text added: "v3.0 (apple IIc)"
- board text removed: "24/04/2026"
- board text removed: "no slot clock"
